Commit message: feat(sim): integrate Gazebo Harmonic, ros_gz_bridge, and 3D LiDAR mapping
- Replace legacy Gazebo Classic stack with Gazebo Harmonic (Gz Sim) on ROS 2 Lyrical
- Add ros_gz_bridge for /clock, /NX01/imu, and GPU LiDAR point clouds (/NX01/mid360_PointCloud2)
- Update quadrotor URDF with native gpu_lidar sensor matching mighty_lyrical_ws architecture
- Modernize fake_sim to teleport UAV pose via ros_gz_interfaces/srv/SetEntityPose
- Add native Gazebo Harmonic SDF 1.8 worlds (easy_forest, medium_forest, hard_forest, ring_forest, etc.)
- Update global_mapper_ros launcher with sim_uav.yaml parameters and Gazebo sim time
- Configure RViz2 view to automatically track the drone in 3D flight (Target Frame: NX01/base_link)
- Add stop_sim.sh and --kill flag in run_sim.py for clean simulation teardown
- Update README.md with Gazebo Harmonic usage and simulation termination commands

File: src/sando/urdf/quadrotor.urdf.xacro (robot description, xacro)
@@ -11,9 +11,55 @@
     <xacro:quadrotor_base_macro />
     <!-- Note: added $(arg namespace)_ to the name to avoid having multiple sensors with the same name when using multiple agents -->
-    <!-- Livox -->
-    <xacro:include filename="$(find ros2_livox_simulation)/urdf/mid360.xacro" />
-    <xacro:mid360 name="$(arg namespace)_livox" namespace="$(arg namespace)" parent="base_link" topic="mid360" >
+    <!-- Livox Mid-360 LiDAR link & joint -->
+    <link name="$(arg namespace)_livox">
+      <inertial>
+        <mass value="0.1" />
+        <origin xyz="0 0 0" rpy="0 0 0" />
+        <inertia ixx="0.0001" ixy="0" ixz="0" iyy="0.0001" iyz="0" izz="0.0001" />
+      </inertial>
+      <visual>
+        <origin xyz="0 0 0" rpy="0 0 0" />
+        <geometry>
+          <cylinder radius="0.04" length="0.06"/>
+        </geometry>
+      </visual>
+    </link>
+    <joint name="$(arg namespace)_livox_joint" type="fixed">
       <origin xyz="0 0 0.2" rpy="0 0.3 0"/>
-    </xacro:mid360>
+      <parent link="base_link"/>
+      <child link="$(arg namespace)_livox"/>
+    </joint>
+    <!-- Native Gz Sim GPU LiDAR (Mid-360 equivalent) -->
+    <gazebo reference="$(arg namespace)_livox">
+      <sensor name="gpu_lidar" type="gpu_lidar">
+        <pose relative_to="$(arg namespace)_livox">0 0 0 0 0 0</pose>
+        <topic>/$(arg namespace)/lidar</topic>
+        <update_rate>10</update_rate>
+        <always_on>true</always_on>
+        <visualize>false</visualize>
+        <gz_frame_id>$(arg namespace)/$(arg namespace)_livox</gz_frame_id>
+        <lidar>
+          <scan>
+            <horizontal>
+              <samples>360</samples>
+              <resolution>1</resolution>
+              <min_angle>-3.14159265359</min_angle>
+              <max_angle>3.14159265359</max_angle>
+            </horizontal>
+            <vertical>
+              <samples>32</samples>
+              <resolution>1</resolution>
+              <min_angle>-0.261799</min_angle>
+              <max_angle>0.785398</max_angle>
+            </vertical>
+          </scan>
+          <range>
+            <min>0.1</min>
+            <max>40.0</max>
+            <resolution>0.01</resolution>
+          </range>
+        </lidar>
+      </sensor>
+    </gazebo>
     <!-- Forward facing camera (d435)-->
     <xacro:include filename="$(find sando)/urdf/_d435.urdf.xacro" />
